File: PCBs/MOL-v2-1_MOD-Actuators.brd (EAGLE design)
At the start: 33 x 43.2 mm, 8 parts, among them IC3 SN74LVC2G04DBV, J1 ACTUATORS, J4 SERVO 1, J5 SERVO 2

Commit message: MOL PCB v2-1 and Modules revisions
Parts:
- moved J5 4.58 mm to (22.9, 8.89)
- moved J4 2.84 mm to (22.9, 11.4)
- moved MOTORS1 2.54 mm to (12.2, 7.62)
Routing:
- net GND: track 62.4 -> 51.6 mm, vias 0 -> 1
- net +5V: track 47.7 -> 37.3 mm
- net +3V3: track 30.3 -> 39.8 mm
- net S2: track 38.7 -> 32.4 mm
- net S1: track 35.3 -> 32.7 mm
- net VMOT: track 23.9 -> 22.0 mm
- net N$3: track 6.57 -> 7.21 mm
- net N$2: track 6.56 -> 7.19 mm
- net N$4: track 6.58 -> 7.20 mm
- net N$1: track 6.58 -> 7.20 mm
Other:
- board text added: "2017 Ali Momeni @ Pittsburgh"
- board text added: "MOL-v2-1 Actuators Module"
